Commit message: Fixed the order of the gripper's functions - need to fix collisions while gripping

File: RobotSimulator_v1/cube_small.urdf (robot description, URDF)
Before this commit: robot cuboid, 1 links, 0 joints
Links:
- link body: geometry collision box size=0.04 0.04 0.04; visual box size=0.04 0.04 0.04

Commit message: Changed the cube to prepare for easier grasp

File: RobotSimulator_v1/cube_small.urdf (robot description, URDF)
Before this commit: robot cuboid, 1 links, 0 joints
Links:
- removed link body
- added link baseLink, mass 0.1; collision box size=.05 .05 .05; visual mesh filename=cube.obj scale=.05 .05 .05
